File: DIN41612_BACKPLANE/DIN41612_BACKPLANE.kicad_pcb (KiCad board)
At the start: 4 copper layers, 299.7 x 128.5 mm, 34 parts, among them J1 615008138221, J10 5535090-4, J11 5535090-4, J12 5535090-4, J13 5535090-4, J14 71918-150LF, J15 1829170, J2 615008138221, J3 615008138221, J4 615008138221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

Commit message: Added trigger signal.
Connections:
- J10 pad A16: (no net) -> /TRG_SIG
- J10 pad C16: (no net) -> /TRG_GND
- J11 pad A16: (no net) -> /TRG_SIG
- J11 pad C16: (no net) -> /TRG_GND
- J12 pad A16: (no net) -> /TRG_SIG
- J12 pad C16: (no net) -> /TRG_GND
- J13 pad A16: (no net) -> /TRG_SIG
- J13 pad C16: (no net) -> /TRG_GND
- J14 pad 31: (no net) -> /TRG_SIG
- J14 pad 32: (no net) -> /TRG_SIG
- J14 pad 33: (no net) -> /TRG_GND
- J14 pad 34: (no net) -> /TRG_GND
- J5 pad 31: (no net) -> /TRG_SIG
- J5 pad 32: (no net) -> /TRG_SIG
- J5 pad 33: (no net) -> /TRG_GND
- J5 pad 34: (no net) -> /TRG_GND
- J8 pad A16: (no net) -> /TRG_SIG
- J8 pad C16: (no net) -> /TRG_GND
- J9 pad A16: (no net) -> /TRG_SIG
- J9 pad C16: (no net) -> /TRG_GND
Routing:
- net /TRG_GND: track 0.00 -> 291.6 mm
- net /TRG_SIG: track 0.00 -> 287.0 mm

Commit message: Fixed bug in PCB.
Routing:
- net /TX6-: track 11.1 -> 9.12 mm
- net /TX5-: track 11.1 -> 9.12 mm
- net /TX3-: track 11.1 -> 9.12 mm
- net /TX1-: track 11.1 -> 9.12 mm
- net /TX4-: track 11.1 -> 9.12 mm
- net /TX2-: track 11.1 -> 9.12 mm
- net /RX1+: track 17.8 -> 16.1 mm
- net /RX2-: track 12.5 -> 14.1 mm
- net /RX4-: track 12.5 -> 14.1 mm
- net /RX5-: track 12.5 -> 14.1 mm
- net /RX3-: track 12.5 -> 14.1 mm
- net /RX6-: track 12.5 -> 14.1 mm
- net /RX6+: track 17.3 -> 16.1 mm
- net /RX4+: track 17.3 -> 16.1 mm
- net /RX2+: track 17.3 -> 16.1 mm
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Other:
- board text added: "DIN 41612 BACKPLANE V1.00 2019"

Commit message: kicad
Routing:
- added copper zone on In2.Cu, net +24V
- added copper zone on In1.Cu, net GND1
- added copper zone on In2.Cu, net GND1
- added copper zone on In1.Cu, net GND2
- added copper zone on In2.Cu, net GND2
- added copper zone on In1.Cu, net GND3
- added copper zone on In2.Cu, net GND3
- added copper zone on In1.Cu, net GND4
- added copper zone on In2.Cu, net GND4
- added copper zone on In1.Cu, net GND5
- added copper zone on In2.Cu, net GND5
- added copper zone on In1.Cu, net GND6
- added copper zone on In2.Cu, net GND6
- added copper zone on In1.Cu, net GNDPWR
- added copper zone on In2.Cu, net GNDPWR
- removed copper zone on Power, net +24V
- removed copper zone on Power, net GND1
- removed copper zone on Signal, net GND1
- removed copper zone on Power, net GND2
- removed copper zone on Signal, net GND2
- removed copper zone on Power, net GND3
- removed copper zone on Signal, net GND3
- removed copper zone on Power, net GND4
- removed copper zone on Signal, net GND4
- removed copper zone on Power, net GND5
- removed copper zone on Signal, net GND5
- removed copper zone on Power, net GND6
- removed copper zone on Signal, net GND6
- removed copper zone on Power, net GNDPWR
- removed copper zone on Signal, net GNDPWR
Other:
- net class Default removed
- net class Signal removed
